Commit message: migrate custom settings in v1.0

File: assistive_gym/envs/assets/wheelchair/wheelchair.urdf (robot description, URDF)
Before this commit: robot wheelchair, 1 links, 0 joints
Links:
- link root: geometry visual mesh filename=wheelchair_permobil_reduced_compressed.obj scale=0.15 0.15 0.15
